File: board/board.kicad_pcb (KiCad board)
At the start: 2 copper layers, 21 x 13 mm, 1 part

Commit message: v1.0
Parts:
- added C1: 100nF, Capacitor_SMD:C_0603_1608Metric, F.Cu at (179.8, 90.8)
- added C10: 100nF, Capacitor_SMD:C_0603_1608Metric, F.Cu at (179.8, 102.2)
- added C11: 100nF, Capacitor_SMD:C_0603_1608Metric, F.Cu at (175.9, 102.2)
- added C12: 100nF, Capacitor_SMD:C_0603_1608Metric, F.Cu at (171.1, 95.4)
- added C13: 2.2uF, Capacitor_SMD:C_0603_1608Metric, F.Cu at (157.2, 92.1)
- added C14: 2.2uF, Capacitor_SMD:C_0603_1608Metric, F.Cu at (172.7, 91.6)
- added C15: 100nF, Capacitor_SMD:C_0603_1608Metric, F.Cu at (150.0, 92.1)
- added C16: 1uF, Capacitor_SMD:C_0603_1608Metric, F.Cu at (148.5, 92.1)
- added C17: 10uF, Capacitor_SMD:C_0603_1608Metric, F.Cu at (169.1, 98.6)
- added C18: 1uF, Capacitor_SMD:C_0603_1608Metric, F.Cu at (155.7, 92.1)
- added C19: 100pF, Capacitor_SMD:C_0402_1005Metric, F.Cu at (158.4, 93.4)
- added C2: 12pF, Capacitor_SMD:C_0603_1608Metric, F.Cu at (188.4, 101.0)
- added C3: 100nF, Capacitor_SMD:C_0603_1608Metric, F.Cu at (171.2, 91.6)
- added C4: 12pF, Capacitor_SMD:C_0603_1608Metric, F.Cu at (183.3, 101.0)
- added C5: 100nF, Capacitor_SMD:C_0603_1608Metric, F.Cu at (184.4, 95.8)
- added C6: 100nF, Capacitor_SMD:C_0603_1608Metric, F.Cu at (184.4, 94.3)
- added C7: 1nF, Capacitor_SMD:C_0603_1608Metric, F.Cu at (184.4, 92.3)
- added C8: 100nF, Capacitor_SMD:C_0603_1608Metric, F.Cu at (175.1, 90.8)
- added C9: 2.2uF, Capacitor_SMD:C_0603_1608Metric, F.Cu at (169.7, 91.6)
- added J1: USB4105-GF-A, b051:GCT_USB4105-GF-A, F.Cu at (162.3, 100.5)
- added J2: 100_digital_IO, on_edge:on_edge_2x05_device, F.Cu at (140.0, 96.5)
- added J3: SWD_6_Pol_Needle, c003:SWD6pol, F.Cu at (190.5, 93.4)
- added J4: 100_digital_IO, on_edge:on_edge_2x05_host, F.Cu at (201.0, 96.5)
- added R2: 10k, Resistor_SMD:R_0603_1608Metric, F.Cu at (184.4, 90.8)
- added R3: 1k, Resistor_SMD:R_0603_1608Metric, F.Cu at (184.5, 97.3)
- added R6: 5.1k, Resistor_SMD:R_0402_1005Metric, F.Cu at (162.0, 93.2)
- added R7: 5.1k, Resistor_SMD:R_0402_1005Metric, F.Cu at (165.2, 94.3)
- added R8: 27R, Resistor_SMD:R_0603_1608Metric, F.Cu at (166.4, 93.0)
- added R9: 27R, Resistor_SMD:R_0603_1608Metric, F.Cu at (166.4, 91.5)
- added U1: W25Q16JVUXIQ, Package_DFN_QFN:DFN-8-1EP_3x2mm_P0.5mm_EP1.3x1.5mm, F.Cu at (171.2, 99.2)
- added U2: RP2040, Package_DFN_QFN:QFN-56-1EP_7x7mm_P0.4mm_EP3.2x3.2mm, F.Cu at (177.8, 96.1)
- added U3: TLV743P, Package_TO_SOT_SMD:SOT-23-5, F.Cu at (152.8, 92.3)
- added Y1: 12MhZ, Crystal:Crystal_SMD_Abracon_ABM8G-4Pin_3.2x2.5mm, F.Cu at (185.8, 100.4)
- moved LOGO1 1.36 mm to (149.2, 97.9)
Routing:
- net GND: track 0.00 -> 171.6 mm, vias 0 -> 36
- net +3V3: track 0.00 -> 150.1 mm, vias 0 -> 11
- net +5V: track 0.00 -> 87.1 mm, vias 0 -> 4
- net /rp2040/~{SPI0_CS}: track 0.00 -> 67.3 mm, vias 0 -> 1
- net /rp2040/SPI0_TX: track 0.00 -> 63.9 mm, vias 0 -> 3
- net /rp2040/GPIO7: track 0.00 -> 63.4 mm, vias 0 -> 1
- net /rp2040/GPIO6: track 0.00 -> 61.7 mm, vias 0 -> 5
- net /rp2040/UART1_TX: track 0.00 -> 60.6 mm, vias 0 -> 1
- net /rp2040/SPI0_RX: track 0.00 -> 60.3 mm, vias 0 -> 3
- net /rp2040/SPI0_SCK: track 0.00 -> 58.8 mm, vias 0 -> 3
- net Net-(C19-Pad1): track 0.00 -> 19.6 mm
- net Net-(U2-VREG_VOUT): track 0.00 -> 19.2 mm, vias 0 -> 3
- net /rp2040/SWCLK: track 0.00 -> 17.5 mm, vias 0 -> 2
- net /rp2040/SWD: track 0.00 -> 16.7 mm, vias 0 -> 2
- net /rp2040/RUN: track 0.00 -> 12.6 mm
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- added copper zone on B.Cu, net GND
- added copper zone on F.Cu, net GND
Other:
- board size 21 x 13 mm -> 61 x 13 mm
- board text added: "osf.100"
- board text added: "osf.c003.v1.0"
